Commit message: fix(system): resolve root causes for symptoms 1, 2, 3 and add soak testing harness

File: src/wh_description/urdf/sensors.xacro (robot description, xacro)
@@ -209,11 +209,11 @@
     <parent link="tool_link"/>
     <child link="hand_camera_link"/>
-    <!-- Gắn tại tâm đế kẹp trùng trục với đầu hút TCP, nhìn vuông góc thẳng xuống dưới -->
-    <origin xyz="0 0 -0.042" rpy="0 1.57079632679 0"/>
+    <!-- Gắn lùi về sau 4cm (-x) trên đế kẹp, nhìn vuông góc thẳng xuống dưới (-z tool_link) -->
+    <origin xyz="-0.040 0.0 -0.042" rpy="0 1.57079632679 0"/>
   </joint>
   <link name="hand_camera_link">
-    <!-- Ngàm đỡ bắt bulông vào mặt trước đế tay kẹp -->
-    <visual>
-      <origin xyz="-0.008 0 0" rpy="0 0 0"/>
+    <!-- Ngàm đỡ bắt bulông vào mặt sau đế tay kẹp (nằm phía sau sensor) -->
+    <visual>
+      <origin xyz="-0.015 0 0" rpy="0 0 0"/>
       <geometry>
         <box size="0.016 0.032 0.016"/>
@@ -221,7 +221,7 @@
       <material name="cam_bracket"/>
     </visual>
-    <!-- Thân vỏ camera -->
-    <visual>
-      <origin xyz="0.006 0 0" rpy="0 0 0"/>
+    <!-- Thân vỏ camera (nằm phía sau sensor) -->
+    <visual>
+      <origin xyz="-0.005 0 0" rpy="0 0 0"/>
       <geometry>
         <box size="0.020 0.036 0.020"/>
@@ -231,5 +231,5 @@
     <!-- Ống kính nhìn thẳng theo trục quang học -->
     <visual>
-      <origin xyz="0.018 0 0" rpy="0 1.57079632679 0"/>
+      <origin xyz="0.005 0 0" rpy="0 1.57079632679 0"/>
       <geometry>
         <cylinder radius="0.007" length="0.006"/>
@@ -246,5 +246,5 @@
     <parent link="hand_camera_link"/>
     <child link="hand_camera_optical_frame"/>
-    <origin xyz="0 0 0" rpy="-1.57079632679 0 -1.57079632679"/>
+    <origin xyz="0.010 0 0" rpy="-1.57079632679 0 -1.57079632679"/>
   </joint>
   <link name="hand_camera_optical_frame"/>
@@ -253,5 +253,5 @@
     <selfCollide>false</selfCollide>
     <sensor name="hand_camera" type="camera">
-      <pose>0 0 0 0 0 0</pose>
+      <pose>0.010 0 0 0 0 0</pose>
       <always_on>true</always_on>
       <update_rate>30</update_rate>

Commit message: fix(dock_camera): pitch dock camera down 11.5 deg, fix reproj_error_px and soak test task status

File: src/wh_description/urdf/sensors.xacro (robot description, xacro)
@@ -130,6 +130,6 @@
     <parent link="lift_carriage_link"/>
     <child link="dock_camera_link"/>
-    <!-- Tâm quang học đặt tại đỉnh toa trượt: x=0.075, y=0, z=0.040 -->
-    <origin xyz="0.075 0.0 0.040" rpy="0 0 0"/>
+    <!-- Tâm quang học đặt tại đỉnh toa trượt, nghiêng góc 0.20 rad (11.5 deg) để bao quát cả tầng 1 (z=0.11m) và tầng 2 (z=0.36m) -->
+    <origin xyz="0.075 0.0 0.040" rpy="0 0.20 0"/>
   </joint>
   <link name="dock_camera_link">

Commit message: fix(camera_servo): fine-tune dock camera pitch to 0.10 rad and servo retry timeout

File: src/wh_description/urdf/sensors.xacro (robot description, xacro)
@@ -130,6 +130,6 @@
     <parent link="lift_carriage_link"/>
     <child link="dock_camera_link"/>
-    <!-- Tâm quang học đặt tại đỉnh toa trượt, nghiêng góc 0.20 rad (11.5 deg) để bao quát cả tầng 1 (z=0.11m) và tầng 2 (z=0.36m) -->
-    <origin xyz="0.075 0.0 0.040" rpy="0 0.20 0"/>
+    <!-- Tâm quang học đặt tại đỉnh toa trượt, nghiêng góc 0.10 rad (5.7 deg) để căn giữa hoàn hảo cả tầng 1 (z=0.11m) và tầng 2 (z=0.36m) -->
+    <origin xyz="0.075 0.0 0.040" rpy="0 0.10 0"/>
   </joint>
   <link name="dock_camera_link">

Commit message: fix(dock_camera): align dock camera horizontally 0 rad for symmetric FOV margins

File: src/wh_description/urdf/sensors.xacro (robot description, xacro)
@@ -130,6 +130,6 @@
     <parent link="lift_carriage_link"/>
     <child link="dock_camera_link"/>
-    <!-- Tâm quang học đặt tại đỉnh toa trượt, nghiêng góc 0.10 rad (5.7 deg) để căn giữa hoàn hảo cả tầng 1 (z=0.11m) và tầng 2 (z=0.36m) -->
-    <origin xyz="0.075 0.0 0.040" rpy="0 0.10 0"/>
+    <!-- Tâm quang học đặt tại đỉnh toa trượt (z=0.23m), hướng ngang thẳng trước (0 deg) để căn giữa đối xứng hoàn hảo cả tầng 1 (z=0.11m, dZ=-0.12m) và tầng 2 (z=0.36m, dZ=+0.13m) -->
+    <origin xyz="0.075 0.0 0.040" rpy="0 0 0"/>
   </joint>
   <link name="dock_camera_link">
