Commit message: Initial commit: warehouse workspace setup

File: src/wh_description/urdf/arm.xacro (robot description, xacro)
@@ -216,15 +216,15 @@
       <material name="arm_hub_mat"/>
     </visual>
-    <!-- Thân đòn cánh tay 2 (dài 0.18 m) -->
-    <visual>
-      <origin xyz="0.09 0 0.013" rpy="0 0 0"/>
-      <geometry>
-        <box size="0.18 0.038 0.026"/>
+    <!-- Thân đòn cánh tay 2 (dài 0.14 m kết hợp ngàm kẹp ngang vươn ra 0.04 m -> tổng tâm kẹp đúng 0.18 m) -->
+    <visual>
+      <origin xyz="0.07 0 0.013" rpy="0 0 0"/>
+      <geometry>
+        <box size="0.14 0.038 0.026"/>
       </geometry>
       <material name="arm_link_color"/>
     </visual>
-    <!-- Trụ cổ tay (Wrist Housing) đâm xuống dưới để nhận đế kẹp -->
-    <visual>
-      <origin xyz="0.18 0 0.005" rpy="0 0 0"/>
+    <!-- Trụ cổ tay (Wrist Housing) nhận khớp nối tay kẹp bẻ ngang -->
+    <visual>
+      <origin xyz="0.14 0 0.005" rpy="0 0 0"/>
       <geometry>
         <cylinder radius="0.022" length="0.036"/>
@@ -233,5 +233,5 @@
     </visual>
     <collision>
-      <origin xyz="0.09 0 0.013" rpy="0 0 0"/>
+      <origin xyz="0.07 0 0.013" rpy="0 0 0"/>
       <geometry>
         <box size="0.14 0.035 0.024"/>
@@ -239,7 +239,7 @@
     </collision>
     <inertial>
-      <origin xyz="0.09 0 0.013" rpy="0 0 0"/>
+      <origin xyz="0.07 0 0.013" rpy="0 0 0"/>
       <mass value="0.35"/>
-      <xacro:box_inertia m="0.35" x="0.18" y="0.038" z="0.026"/>
+      <xacro:box_inertia m="0.35" x="0.14" y="0.038" z="0.026"/>
     </inertial>
   </link>
@@ -249,19 +249,26 @@
   </gazebo>
   <!-- ======================================================== -->
-  <!-- 5. TAY KẸP CƠ KHÍ 2 NGÓN (PARALLEL GRIPPER)               -->
-  <!-- ======================================================== -->
-  <!-- Khớp gắn đế kẹp cắm khít vào đáy trụ cổ tay của cánh tay 2 -->
-  <joint name="tool_joint" type="fixed">
+  <!-- 5. TAY KẸP CƠ KHÍ 2 NGÓN BẺ NGANG (HORIZONTAL GRIPPER)    -->
+  <!-- ======================================================== -->
+  <!-- Khớp cổ tay xoay (Revolute Wrist Joint) kết nối cánh tay 2 với đế tay kẹp -->
+  <joint name="wrist_joint" type="revolute">
     <parent link="elbow_link"/>
     <child link="tool_link"/>
-    <origin xyz="0.18 0 -0.013" rpy="0 0 0"/>
-  </joint>
-  <!-- Thân đế tay kẹp (Gripper Base / Palm) -->
+    <origin xyz="0.14 0 -0.013" rpy="0 0 0"/>
+    <axis xyz="0 0 1"/>
+    <limit lower="-3.141592653589793" upper="3.141592653589793" effort="30.0" velocity="2.0"/>
+    <dynamics damping="0.5" friction="0.1"/>
+  </joint>
+  <gazebo reference="wrist_joint">
+    <implicitSpringDamper>true</implicitSpringDamper>
+    <provideFeedback>true</provideFeedback>
+  </gazebo>
+  <!-- Thân đế tay kẹp bẻ ngang (Horizontal Gripper Base / Palm) -->
   <link name="tool_link">
-    <!-- Trụ cổ kẹp cắm trực tiếp vào cổ tay -->
-    <visual>
-      <origin xyz="0 0 -0.018" rpy="0 0 0"/>
-      <geometry>
-        <cylinder radius="0.014" length="0.036"/>
+    <!-- Cổ trụ đứng thả từ cổ tay xuống cao độ thao tác -->
+    <visual>
+      <origin xyz="0 0 -0.028" rpy="0 0 0"/>
+      <geometry>
+        <cylinder radius="0.014" length="0.056"/>
       </geometry>
       <material name="gripper_stem_mat">
@@ -269,9 +276,9 @@
       </material>
     </visual>
-    <!-- Thanh ngang thân đế kẹp -->
-    <visual>
-      <origin xyz="0 0 -0.042" rpy="0 0 0"/>
-      <geometry>
-        <box size="0.045 0.096 0.014"/>
+    <!-- Khớp khuỷu adapter bẻ 90 độ sang ngang vươn về phía trước (+x) -->
+    <visual>
+      <origin xyz="0.008 0 -0.056" rpy="0 0 0"/>
+      <geometry>
+        <box size="0.022 0.032 0.020"/>
       </geometry>
       <material name="gripper_palm_mat">
@@ -279,29 +286,37 @@
       </material>
     </visual>
-    <!-- Bulông chốt má kẹp hai bên -->
-    <visual>
-      <origin xyz="0 0.038 -0.049" rpy="0 0 0"/>
-      <geometry>
-        <cylinder radius="0.008" length="0.006"/>
+    <!-- Mặt bích đế kẹp dựng đứng hướng mặt về phía trước (+x) -->
+    <visual>
+      <origin xyz="0.018 0 -0.056" rpy="0 0 0"/>
+      <geometry>
+        <box size="0.008 0.096 0.038"/>
+      </geometry>
+      <material name="gripper_palm_mat"/>
+    </visual>
+    <!-- Bulông chốt má kẹp hai bên nằm ngang -->
+    <visual>
+      <origin xyz="0.014 0.038 -0.056" rpy="0 1.5707963 0"/>
+      <geometry>
+        <cylinder radius="0.007" length="0.012"/>
       </geometry>
       <material name="gripper_stem_mat"/>
     </visual>
     <visual>
-      <origin xyz="0 -0.038 -0.049" rpy="0 0 0"/>
-      <geometry>
-        <cylinder radius="0.008" length="0.006"/>
+      <origin xyz="0.014 -0.038 -0.056" rpy="0 1.5707963 0"/>
+      <geometry>
+        <cylinder radius="0.007" length="0.012"/>
       </geometry>
       <material name="gripper_stem_mat"/>
     </visual>
     <collision>
-      <origin xyz="0 0 -0.042" rpy="0 0 0"/>
-      <geometry>
-        <box size="0.045 0.096 0.014"/>
-      </geometry>
-    </collision>
-    <inertial>
-      <origin xyz="0 0 -0.035" rpy="0 0 0"/>
+      <origin xyz="0.008 0 -0.056" rpy="0 0 0"/>
+      <geometry>
+        <box size="0.024 0.096 0.038"/>
+      </geometry>
+    </collision>
+    <inertial>
+      <origin xyz="0.008 0 -0.045" rpy="0 0 0"/>
       <mass value="0.25"/>
-      <xacro:box_inertia m="0.25" x="0.045" y="0.096" z="0.035"/>
+      <xacro:box_inertia m="0.25" x="0.030" y="0.096" z="0.050"/>
     </inertial>
   </link>
@@ -311,18 +326,18 @@
   </gazebo>
   <!-- ======================================================== -->
-  <!-- 6. HAI MÁ KẸP SONG SONG (PARALLEL FINGERS)               -->
-  <!-- ======================================================== -->
-  <!-- Má kẹp trái (Left Finger) gắn liền dưới đế kẹp -->
+  <!-- 6. HAI MÁ KẸP SONG SONG BẺ NGANG (HORIZONTAL FINGERS)    -->
+  <!-- ======================================================== -->
+  <!-- Má kẹp trái (Left Finger) vươn ngang về phía trước (+x) -->
   <joint name="left_finger_joint" type="fixed">
     <parent link="tool_link"/>
     <child link="left_finger_link"/>
-    <origin xyz="0 0.038 -0.049" rpy="0 0 0"/>
+    <origin xyz="0.022 0.038 -0.056" rpy="0 0 0"/>
   </joint>
   <link name="left_finger_link">
-    <!-- Khung ngón kẹp kim loại -->
-    <visual>
-      <origin xyz="0 0 -0.021" rpy="0 0 0"/>
-      <geometry>
-        <box size="0.036 0.010 0.042"/>
+    <!-- Khung ngón kẹp kim loại vươn ngang ra -->
+    <visual>
+      <origin xyz="0.022 0 0" rpy="0 0 0"/>
+      <geometry>
+        <box size="0.044 0.010 0.028"/>
       </geometry>
       <material name="finger_metal_mat">
@@ -330,9 +345,9 @@
       </material>
     </visual>
-    <!-- Đệm cao su ma sát cao màu cam phía trong lòng ngón kẹp -->
-    <visual>
-      <origin xyz="0 -0.0055 -0.021" rpy="0 0 0"/>
-      <geometry>
-        <box size="0.032 0.0025 0.038"/>
+    <!-- Đệm cao su ma sát cao màu cam phía trong lòng ngón kẹp (hướng vào -y) -->
+    <visual>
+      <origin xyz="0.022 -0.0055 0" rpy="0 0 0"/>
+      <geometry>
+        <box size="0.040 0.0025 0.024"/>
       </geometry>
       <material name="rubber_pad_mat">
@@ -341,13 +356,13 @@
     </visual>
     <collision>
-      <origin xyz="0 0 -0.021" rpy="0 0 0"/>
-      <geometry>
-        <box size="0.036 0.010 0.042"/>
-      </geometry>
-    </collision>
-    <inertial>
-      <origin xyz="0 0 -0.021" rpy="0 0 0"/>
+      <origin xyz="0.022 0 0" rpy="0 0 0"/>
+      <geometry>
+        <box size="0.044 0.010 0.028"/>
+      </geometry>
+    </collision>
+    <inertial>
+      <origin xyz="0.022 0 0" rpy="0 0 0"/>
       <mass value="0.05"/>
-      <xacro:box_inertia m="0.05" x="0.036" y="0.010" z="0.042"/>
+      <xacro:box_inertia m="0.05" x="0.044" y="0.010" z="0.028"/>
     </inertial>
   </link>
@@ -358,37 +373,37 @@
     <selfCollide>false</selfCollide>
   </gazebo>
-  <!-- Má kẹp phải (Right Finger) gắn liền dưới đế kẹp -->
+  <!-- Má kẹp phải (Right Finger) vươn ngang về phía trước (+x) -->
   <joint name="right_finger_joint" type="fixed">
     <parent link="tool_link"/>
     <child link="right_finger_link"/>
-    <origin xyz="0 -0.038 -0.049" rpy="0 0 0"/>
+    <origin xyz="0.022 -0.038 -0.056" rpy="0 0 0"/>
   </joint>
   <link name="right_finger_link">
-    <!-- Khung ngón kẹp kim loại -->
-    <visual>
-      <origin xyz="0 0 -0.021" rpy="0 0 0"/>
-      <geometry>
-        <box size="0.036 0.010 0.042"/>
+    <!-- Khung ngón kẹp kim loại vươn ngang ra -->
+    <visual>
+      <origin xyz="0.022 0 0" rpy="0 0 0"/>
+      <geometry>
+        <box size="0.044 0.010 0.028"/>
       </geometry>
       <material name="finger_metal_mat"/>
     </visual>
-    <!-- Đệm cao su ma sát cao màu cam phía trong lòng ngón kẹp -->
-    <visual>
-      <origin xyz="0 0.0055 -0.021" rpy="0 0 0"/>
-      <geometry>
-        <box size="0.032 0.0025 0.038"/>
+    <!-- Đệm cao su ma sát cao màu cam phía trong lòng ngón kẹp (hướng vào +y) -->
+    <visual>
+      <origin xyz="0.022 0.0055 0" rpy="0 0 0"/>
+      <geometry>
+        <box size="0.040 0.0025 0.024"/>
       </geometry>
       <material name="rubber_pad_mat"/>
     </visual>
     <collision>
-      <origin xyz="0 0 -0.021" rpy="0 0 0"/>
-      <geometry>
-        <box size="0.036 0.010 0.042"/>
-      </geometry>
-    </collision>
-    <inertial>
-      <origin xyz="0 0 -0.021" rpy="0 0 0"/>
+      <origin xyz="0.022 0 0" rpy="0 0 0"/>
+      <geometry>
+        <box size="0.044 0.010 0.028"/>
+      </geometry>
+    </collision>
+    <inertial>
+      <origin xyz="0.022 0 0" rpy="0 0 0"/>
       <mass value="0.05"/>
-      <xacro:box_inertia m="0.05" x="0.036" y="0.010" z="0.042"/>
+      <xacro:box_inertia m="0.05" x="0.044" y="0.010" z="0.028"/>
     </inertial>
   </link>
@@ -402,9 +417,10 @@
   <!-- 7. TÂM KẸP (TCP - TOOL CENTER POINT) & GRASP LINK         -->
   <!-- ======================================================== -->
-  <!-- Điểm tâm kẹp nằm chính giữa 2 má kẹp (z = -0.070 m từ tool_link) -->
+  <!-- Điểm tâm kẹp nằm chính giữa 2 má kẹp (x = 0.040 m, z = -0.056 m từ tool_link) -->
+  <!-- Tổng tầm vươn khâu 2 đến tâm kẹp: 0.14 m + 0.04 m = 0.180 m chuẩn xác -->
   <joint name="gripper_grasp_joint" type="fixed">
     <parent link="tool_link"/>
     <child link="gripper_grasp_link"/>
-    <origin xyz="0 0 -0.070" rpy="0 0 0"/>
+    <origin xyz="0.040 0 -0.056" rpy="0 0 0"/>
   </joint>
   <link name="gripper_grasp_link">

File: src/wh_description/urdf/base.xacro (robot description, xacro)
@@ -38,4 +38,5 @@
     <kp>1000000.0</kp>
     <kd>1.0</kd>
+    <selfCollide>false</selfCollide>
   </gazebo>
   <!-- ======================================================== -->
@@ -151,9 +152,9 @@
   </joint>
   <link name="tray_link">
-    <!-- Đáy khay đựng hàng (kích thước 12x12 cm vừa vặn cho hộp 6x6 cm) -->
+    <!-- Đáy khay đựng hàng (kích thước mở rộng 15x15 cm rộng rãi cho hộp 6x6 cm) -->
     <visual>
       <origin xyz="0 0 0.003" rpy="0 0 0"/>
       <geometry>
-        <box size="0.12 0.12 0.006"/>
+        <box size="0.15 0.15 0.006"/>
       </geometry>
       <material name="tray_body_mat">
@@ -165,5 +166,5 @@
       <origin xyz="0 0 0.0065" rpy="0 0 0"/>
       <geometry>
-        <box size="0.108 0.108 0.002"/>
+        <box size="0.138 0.138 0.002"/>
       </geometry>
       <material name="tray_mat_rubber">
@@ -171,66 +172,100 @@
       </material>
     </visual>
-    <!-- Thành trước khay (Front Lip) -->
-    <visual>
-      <origin xyz="0.057 0 0.012" rpy="0 0 0"/>
-      <geometry>
-        <box size="0.006 0.12 0.018"/>
-      </geometry>
-      <material name="tray_body_mat"/>
-    </visual>
-    <!-- Thành sau khay (Rear Lip) -->
-    <visual>
-      <origin xyz="-0.057 0 0.012" rpy="0 0 0"/>
-      <geometry>
-        <box size="0.006 0.12 0.018"/>
-      </geometry>
-      <material name="tray_body_mat"/>
-    </visual>
-    <!-- Thành trái khay (Left Wall) -->
-    <visual>
-      <origin xyz="0 0.057 0.012" rpy="0 0 0"/>
-      <geometry>
-        <box size="0.108 0.006 0.018"/>
-      </geometry>
-      <material name="tray_body_mat"/>
-    </visual>
-    <!-- Thành phải khay (Right Wall) -->
-    <visual>
-      <origin xyz="0 -0.057 0.012" rpy="0 0 0"/>
-      <geometry>
-        <box size="0.108 0.006 0.018"/>
-      </geometry>
-      <material name="tray_body_mat"/>
-    </visual>
-    <!-- Viền phản quang an toàn màu cam trên miệng khay -->
-    <visual>
-      <origin xyz="0 0.057 0.0215" rpy="0 0 0"/>
-      <geometry><box size="0.12 0.008 0.002"/></geometry>
+    <!-- Thành trước khay (Front Wall - Cao 16mm chuẩn AMR, giữ hộp nhưng không cản trở tay kẹp) -->
+    <visual>
+      <origin xyz="0.072 0 0.014" rpy="0 0 0"/>
+      <geometry>
+        <box size="0.006 0.15 0.016"/>
+      </geometry>
+      <material name="tray_body_mat"/>
+    </visual>
+    <!-- Thành sau khay (Rear Wall - Cao 16mm) -->
+    <visual>
+      <origin xyz="-0.072 0 0.014" rpy="0 0 0"/>
+      <geometry>
+        <box size="0.006 0.15 0.016"/>
+      </geometry>
+      <material name="tray_body_mat"/>
+    </visual>
+    <!-- Thành trái khay (Left Wall - Cao 16mm) -->
+    <visual>
+      <origin xyz="0 0.072 0.014" rpy="0 0 0"/>
+      <geometry>
+        <box size="0.138 0.006 0.016"/>
+      </geometry>
+      <material name="tray_body_mat"/>
+    </visual>
+    <!-- Thành phải khay (Right Wall - Cao 16mm) -->
+    <visual>
+      <origin xyz="0 -0.072 0.014" rpy="0 0 0"/>
+      <geometry>
+        <box size="0.138 0.006 0.016"/>
+      </geometry>
+      <material name="tray_body_mat"/>
+    </visual>
+    <!-- Viền phản quang an toàn màu cam trên đỉnh 4 thành khay -->
+    <visual>
+      <origin xyz="0.072 0 0.023" rpy="0 0 0"/>
+      <geometry><box size="0.008 0.15 0.002"/></geometry>
       <material name="tray_rim_mat"><color rgba="0.95 0.45 0.10 1.0"/></material>
     </visual>
     <visual>
-      <origin xyz="0 -0.057 0.0215" rpy="0 0 0"/>
-      <geometry><box size="0.12 0.008 0.002"/></geometry>
+      <origin xyz="-0.072 0 0.023" rpy="0 0 0"/>
+      <geometry><box size="0.008 0.15 0.002"/></geometry>
       <material name="tray_rim_mat"/>
     </visual>
-    <!-- Collision day khay (chi giu collision mat day de do hop, khong de thanh khay va quet tay kep) -->
+    <visual>
+      <origin xyz="0 0.072 0.023" rpy="0 0 0"/>
+      <geometry><box size="0.138 0.008 0.002"/></geometry>
+      <material name="tray_rim_mat"/>
+    </visual>
+    <visual>
+      <origin xyz="0 -0.072 0.023" rpy="0 0 0"/>
+      <geometry><box size="0.138 0.008 0.002"/></geometry>
+      <material name="tray_rim_mat"/>
+    </visual>
+    <!-- Collision: Đáy khay + 4 gờ chặn chống trượt cao 16mm (thấp hơn hộp 40mm giúp tay kẹp ngang ôm hộp 100% tự do) -->
     <collision>
       <origin xyz="0 0 0.003" rpy="0 0 0"/>
       <geometry>
-        <box size="0.12 0.12 0.006"/>
+        <box size="0.15 0.15 0.006"/>
+      </geometry>
+    </collision>
+    <collision>
+      <origin xyz="0.072 0 0.014" rpy="0 0 0"/>
+      <geometry>
+        <box size="0.006 0.15 0.016"/>
+      </geometry>
+    </collision>
+    <collision>
+      <origin xyz="-0.072 0 0.014" rpy="0 0 0"/>
+      <geometry>
+        <box size="0.006 0.15 0.016"/>
+      </geometry>
+    </collision>
+    <collision>
+      <origin xyz="0 0.072 0.014" rpy="0 0 0"/>
+      <geometry>
+        <box size="0.138 0.006 0.016"/>
+      </geometry>
+    </collision>
+    <collision>
+      <origin xyz="0 -0.072 0.014" rpy="0 0 0"/>
+      <geometry>
+        <box size="0.138 0.006 0.016"/>
       </geometry>
     </collision>
     <inertial>
       <origin xyz="0 0 0.010" rpy="0 0 0"/>
-      <mass value="0.25"/>
-      <xacro:box_inertia m="0.25" x="0.14" y="0.20" z="0.024"/>
+      <mass value="0.30"/>
+      <xacro:box_inertia m="0.30" x="0.15" y="0.15" z="0.024"/>
     </inertial>
   </link>
   <gazebo reference="tray_link">
     <material>Gazebo/DarkGrey</material>
-    <mu1>50.0</mu1>
-    <mu2>50.0</mu2>
+    <mu1>100.0</mu1>
+    <mu2>100.0</mu2>
     <kp>1000000.0</kp>
-    <kd>1.0</kd>
+    <kd>10.0</kd>
     <selfCollide>false</selfCollide>
   </gazebo>

File: src/wh_description/urdf/ros2_control.xacro (robot description, xacro)
@@ -27,4 +27,11 @@
       <state_interface name="velocity"/>
     </joint>
+    <joint name="wrist_joint">
+      <command_interface name="position"/>
+      <state_interface name="position">
+        <param name="initial_value">0.0</param>
+      </state_interface>
+      <state_interface name="velocity"/>
+    </joint>
   </ros2_control>
   <gazebo>

File: src/wh_description/urdf/sensors.xacro (robot description, xacro)
@@ -66,5 +66,5 @@
         </scan>
         <range>
-          <min>0.25</min>
+          <min>0.38</min>
           <max>12.0</max>
           <resolution>0.01</resolution>
@@ -125,11 +125,11 @@
   <!-- ======================================================== -->
   <!-- ======================================================== -->
-  <!-- DOCK CAMERA (Gắn trên toa trượt nâng hạ, nhìn thẳng trước) -->
+  <!-- DOCK CAMERA (Gắn cố định trên thân xe, z=0.23m, nhìn ngang) -->
   <!-- ======================================================== -->
   <joint name="dock_camera_joint" type="fixed">
-    <parent link="lift_carriage_link"/>
+    <parent link="base_link"/>
     <child link="dock_camera_link"/>
-    <!-- Tâm quang học đặt tại đỉnh toa trượt (z=0.23m), hướng ngang thẳng trước (0 deg) để căn giữa đối xứng hoàn hảo cả tầng 1 (z=0.11m, dZ=-0.12m) và tầng 2 (z=0.36m, dZ=+0.13m) -->
-    <origin xyz="0.075 0.0 0.040" rpy="0 0 0"/>
+    <!-- Tâm quang học đặt cố định trên thân xe tại z=0.23m (cách đất), hướng ngang thẳng trước (0 deg) căn giữa đối xứng hoàn hảo cả tầng 1 (z=0.11m, dZ=-0.12m) và tầng 2 (z=0.36m, dZ=+0.13m) -->
+    <origin xyz="0.19 0.0 0.14" rpy="0 0 0"/>
   </joint>
   <link name="dock_camera_link">
@@ -204,11 +204,12 @@
   </gazebo>
   <!-- ======================================================== -->
-  <!-- HAND CAMERA (Gắn trên đế tay kẹp, nhìn vuông góc xuống)  -->
+  <!-- ======================================================== -->
+  <!-- HAND CAMERA (Gắn trên đế tay kẹp bẻ ngang, nhìn về phía trước) -->
   <!-- ======================================================== -->
   <joint name="hand_camera_joint" type="fixed">
     <parent link="tool_link"/>
     <child link="hand_camera_link"/>
-    <!-- Gắn lùi về sau 4cm (-x) trên đế kẹp, nhìn vuông góc thẳng xuống dưới (-z tool_link) -->
-    <origin xyz="-0.040 0.0 -0.042" rpy="0 1.57079632679 0"/>
+    <!-- Gắn trên sống lưng khớp bẻ ngang, nhìn theo phương +X và chúi nhẹ 12.6 độ xuống hộp -->
+    <origin xyz="0.006 0.0 -0.038" rpy="0 0.22 0"/>
   </joint>
   <link name="hand_camera_link">
