Commit message: feat: add station management endpoints, cache control headers, and inventory location code tests

File: src/wh_description/urdf/arm.xacro (robot description, xacro)
@@ -266,9 +266,9 @@
   <!-- Thân đế tay kẹp bẻ ngang (Horizontal Gripper Base / Palm) -->
   <link name="tool_link">
-    <!-- Cổ trụ đứng thả từ cổ tay xuống cao độ thao tác -->
-    <visual>
-      <origin xyz="0 0 -0.028" rpy="0 0 0"/>
-      <geometry>
-        <cylinder radius="0.014" length="0.056"/>
+    <!-- Cổ trụ đứng thả từ cổ tay xuống cao độ thao tác (gọn gàng 70mm, chuẩn tâm hông hộp) -->
+    <visual>
+      <origin xyz="0 0 -0.035" rpy="0 0 0"/>
+      <geometry>
+        <cylinder radius="0.014" length="0.070"/>
       </geometry>
       <material name="gripper_stem_mat">
@@ -278,7 +278,7 @@
     <!-- Khớp khuỷu adapter bẻ 90 độ sang ngang vươn về phía trước (+x) -->
     <visual>
-      <origin xyz="0.008 0 -0.056" rpy="0 0 0"/>
-      <geometry>
-        <box size="0.022 0.032 0.020"/>
+      <origin xyz="0.008 0 -0.070" rpy="0 0 0"/>
+      <geometry>
+        <box size="0.020 0.030 0.018"/>
       </geometry>
       <material name="gripper_palm_mat">
@@ -286,37 +286,52 @@
       </material>
     </visual>
-    <!-- Mặt bích đế kẹp dựng đứng hướng mặt về phía trước (+x) -->
-    <visual>
-      <origin xyz="0.018 0 -0.056" rpy="0 0 0"/>
-      <geometry>
-        <box size="0.008 0.096 0.038"/>
+    <!-- Mặt bích đế kẹp dựng đứng hướng mặt về phía trước (+x), rộng 120mm đỡ chắc chắn 2 má kẹp -->
+    <visual>
+      <origin xyz="0.016 0 -0.070" rpy="0 0 0"/>
+      <geometry>
+        <box size="0.008 0.120 0.028"/>
       </geometry>
       <material name="gripper_palm_mat"/>
     </visual>
+    <!-- Ray trượt kim loại dẫn hướng má kẹp trên và dưới -->
+    <visual>
+      <origin xyz="0.017 0 -0.059" rpy="0 0 0"/>
+      <geometry>
+        <box size="0.003 0.120 0.004"/>
+      </geometry>
+      <material name="gripper_stem_mat"/>
+    </visual>
+    <visual>
+      <origin xyz="0.017 0 -0.081" rpy="0 0 0"/>
+      <geometry>
+        <box size="0.003 0.120 0.004"/>
+      </geometry>
+      <material name="gripper_stem_mat"/>
+    </visual>
     <!-- Bulông chốt má kẹp hai bên nằm ngang -->
     <visual>
-      <origin xyz="0.014 0.038 -0.056" rpy="0 1.5707963 0"/>
-      <geometry>
-        <cylinder radius="0.007" length="0.012"/>
+      <origin xyz="0.014 0.036 -0.070" rpy="0 1.5707963 0"/>
+      <geometry>
+        <cylinder radius="0.006" length="0.010"/>
       </geometry>
       <material name="gripper_stem_mat"/>
     </visual>
     <visual>
-      <origin xyz="0.014 -0.038 -0.056" rpy="0 1.5707963 0"/>
-      <geometry>
-        <cylinder radius="0.007" length="0.012"/>
+      <origin xyz="0.014 -0.036 -0.070" rpy="0 1.5707963 0"/>
+      <geometry>
+        <cylinder radius="0.006" length="0.010"/>
       </geometry>
       <material name="gripper_stem_mat"/>
     </visual>
     <collision>
-      <origin xyz="0.008 0 -0.056" rpy="0 0 0"/>
-      <geometry>
-        <box size="0.024 0.096 0.038"/>
-      </geometry>
-    </collision>
-    <inertial>
-      <origin xyz="0.008 0 -0.045" rpy="0 0 0"/>
-      <mass value="0.25"/>
-      <xacro:box_inertia m="0.25" x="0.030" y="0.096" z="0.050"/>
+      <origin xyz="0.004 0 -0.070" rpy="0 0 0"/>
+      <geometry>
+        <box size="0.012 0.120 0.028"/>
+      </geometry>
+    </collision>
+    <inertial>
+      <origin xyz="0.004 0 -0.055" rpy="0 0 0"/>
+      <mass value="0.20"/>
+      <xacro:box_inertia m="0.20" x="0.020" y="0.120" z="0.040"/>
     </inertial>
   </link>
@@ -328,16 +343,23 @@
   <!-- 6. HAI MÁ KẸP SONG SONG BẺ NGANG (HORIZONTAL FINGERS)    -->
   <!-- ======================================================== -->
-  <!-- Má kẹp trái (Left Finger) vươn ngang về phía trước (+x) -->
-  <joint name="left_finger_joint" type="fixed">
+  <!-- Má kẹp trái (Left Finger) vươn ngang về phía trước (+x), trượt dọc trục Y (prismatic) -->
+  <joint name="left_finger_joint" type="prismatic">
     <parent link="tool_link"/>
     <child link="left_finger_link"/>
-    <origin xyz="0.022 0.038 -0.056" rpy="0 0 0"/>
-  </joint>
+    <origin xyz="0.016 0.036 -0.070" rpy="0 0 0"/>
+    <axis xyz="0 1 0"/>
+    <limit lower="-0.008" upper="0.016" effort="60.0" velocity="0.10"/>
+    <dynamics damping="1.0" friction="0.5"/>
+  </joint>
+  <gazebo reference="left_finger_joint">
+    <implicitSpringDamper>true</implicitSpringDamper>
+    <provideFeedback>true</provideFeedback>
+  </gazebo>
   <link name="left_finger_link">
-    <!-- Khung ngón kẹp kim loại vươn ngang ra -->
-    <visual>
-      <origin xyz="0.022 0 0" rpy="0 0 0"/>
-      <geometry>
-        <box size="0.044 0.010 0.028"/>
+    <!-- Khung ngón kẹp kim loại kéo dài 65mm (ôm trọn >84% chiều dài hộp 60mm, kẹp vững chắc) -->
+    <visual>
+      <origin xyz="0.0325 0 0" rpy="0 0 0"/>
+      <geometry>
+        <box size="0.065 0.008 0.024"/>
       </geometry>
       <material name="finger_metal_mat">
@@ -347,7 +369,7 @@
     <!-- Đệm cao su ma sát cao màu cam phía trong lòng ngón kẹp (hướng vào -y) -->
     <visual>
-      <origin xyz="0.022 -0.0055 0" rpy="0 0 0"/>
-      <geometry>
-        <box size="0.040 0.0025 0.024"/>
+      <origin xyz="0.0325 -0.0045 0" rpy="0 0 0"/>
+      <geometry>
+        <box size="0.060 0.0025 0.020"/>
       </geometry>
       <material name="rubber_pad_mat">
@@ -356,33 +378,44 @@
     </visual>
     <collision>
-      <origin xyz="0.022 0 0" rpy="0 0 0"/>
-      <geometry>
-        <box size="0.044 0.010 0.028"/>
-      </geometry>
-    </collision>
-    <inertial>
-      <origin xyz="0.022 0 0" rpy="0 0 0"/>
-      <mass value="0.05"/>
-      <xacro:box_inertia m="0.05" x="0.044" y="0.010" z="0.028"/>
+      <origin xyz="0.0325 0 0" rpy="0 0 0"/>
+      <geometry>
+        <box size="0.065 0.006 0.024"/>
+      </geometry>
+    </collision>
+    <inertial>
+      <origin xyz="0.0325 0 0" rpy="0 0 0"/>
+      <mass value="0.045"/>
+      <xacro:box_inertia m="0.045" x="0.065" y="0.008" z="0.024"/>
     </inertial>
   </link>
   <gazebo reference="left_finger_link">
     <material>Gazebo/Orange</material>
-    <mu1>2.0</mu1>
-    <mu2>2.0</mu2>
-    <selfCollide>false</selfCollide>
-  </gazebo>
-  <!-- Má kẹp phải (Right Finger) vươn ngang về phía trước (+x) -->
-  <joint name="right_finger_joint" type="fixed">
+    <kp>1000000.0</kp>
+    <kd>100.0</kd>
+    <minDepth>0.002</minDepth>
+    <maxVel>0.01</maxVel>
+    <mu1>50.0</mu1>
+    <mu2>50.0</mu2>
+    <selfCollide>false</selfCollide>
+  </gazebo>
+  <!-- Má kẹp phải (Right Finger) vươn ngang về phía trước (+x), trượt dọc trục Y (prismatic) -->
+  <joint name="right_finger_joint" type="prismatic">
     <parent link="tool_link"/>
     <child link="right_finger_link"/>
-    <origin xyz="0.022 -0.038 -0.056" rpy="0 0 0"/>
-  </joint>
+    <origin xyz="0.016 -0.036 -0.070" rpy="0 0 0"/>
+    <axis xyz="0 1 0"/>
+    <limit lower="-0.016" upper="0.008" effort="60.0" velocity="0.10"/>
+    <dynamics damping="1.0" friction="0.5"/>
+  </joint>
+  <gazebo reference="right_finger_joint">
+    <implicitSpringDamper>true</implicitSpringDamper>
+    <provideFeedback>true</provideFeedback>
+  </gazebo>
   <link name="right_finger_link">
-    <!-- Khung ngón kẹp kim loại vươn ngang ra -->
-    <visual>
-      <origin xyz="0.022 0 0" rpy="0 0 0"/>
-      <geometry>
-        <box size="0.044 0.010 0.028"/>
+    <!-- Khung ngón kẹp kim loại kéo dài 65mm (ôm trọn >84% chiều dài hộp 60mm, kẹp vững chắc) -->
+    <visual>
+      <origin xyz="0.0325 0 0" rpy="0 0 0"/>
+      <geometry>
+        <box size="0.065 0.008 0.024"/>
       </geometry>
       <material name="finger_metal_mat"/>
@@ -390,26 +423,30 @@
     <!-- Đệm cao su ma sát cao màu cam phía trong lòng ngón kẹp (hướng vào +y) -->
     <visual>
-      <origin xyz="0.022 0.0055 0" rpy="0 0 0"/>
-      <geometry>
-        <box size="0.040 0.0025 0.024"/>
+      <origin xyz="0.0325 0.0045 0" rpy="0 0 0"/>
+      <geometry>
+        <box size="0.060 0.0025 0.020"/>
       </geometry>
       <material name="rubber_pad_mat"/>
     </visual>
     <collision>
-      <origin xyz="0.022 0 0" rpy="0 0 0"/>
-      <geometry>
-        <box size="0.044 0.010 0.028"/>
-      </geometry>
-    </collision>
-    <inertial>
-      <origin xyz="0.022 0 0" rpy="0 0 0"/>
-      <mass value="0.05"/>
-      <xacro:box_inertia m="0.05" x="0.044" y="0.010" z="0.028"/>
+      <origin xyz="0.0325 0 0" rpy="0 0 0"/>
+      <geometry>
+        <box size="0.065 0.006 0.024"/>
+      </geometry>
+    </collision>
+    <inertial>
+      <origin xyz="0.0325 0 0" rpy="0 0 0"/>
+      <mass value="0.045"/>
+      <xacro:box_inertia m="0.045" x="0.065" y="0.008" z="0.024"/>
     </inertial>
   </link>
   <gazebo reference="right_finger_link">
     <material>Gazebo/Orange</material>
-    <mu1>2.0</mu1>
-    <mu2>2.0</mu2>
+    <kp>1000000.0</kp>
+    <kd>100.0</kd>
+    <minDepth>0.002</minDepth>
+    <maxVel>0.01</maxVel>
+    <mu1>50.0</mu1>
+    <mu2>50.0</mu2>
     <selfCollide>false</selfCollide>
   </gazebo>
@@ -417,10 +454,9 @@
   <!-- 7. TÂM KẸP (TCP - TOOL CENTER POINT) & GRASP LINK         -->
   <!-- ======================================================== -->
-  <!-- Điểm tâm kẹp nằm chính giữa 2 má kẹp (x = 0.040 m, z = -0.056 m từ tool_link) -->
-  <!-- Tổng tầm vươn khâu 2 đến tâm kẹp: 0.14 m + 0.04 m = 0.180 m chuẩn xác -->
+  <!-- Điểm tâm kẹp nằm chính giữa 2 má kẹp (x = 0.058 m, z = -0.070 m từ tool_link, cách mặt bích 38mm, triệt tiêu 100% va chạm đế) -->
   <joint name="gripper_grasp_joint" type="fixed">
     <parent link="tool_link"/>
     <child link="gripper_grasp_link"/>
-    <origin xyz="0.040 0 -0.056" rpy="0 0 0"/>
+    <origin xyz="0.058 0 -0.070" rpy="0 0 0"/>
   </joint>
   <link name="gripper_grasp_link">

File: src/wh_description/urdf/gazebo_plugins.xacro (robot description, xacro)
@@ -18,7 +18,7 @@
     </plugin>
   </gazebo>
-  <!-- Parallel Gripper Attachment Plugin (Gazebo object attacher) -->
+  <!-- Parallel Gripper Attachment Plugin (Gazebo object attacher with zero vibration) -->
   <gazebo>
-    <plugin name="parallel_gripper" filename="libgazebo_ros_vacuum_gripper.so">
+    <plugin name="parallel_gripper" filename="libwh_gripper_attacher.so">
       <ros>
         <namespace>gripper</namespace>
@@ -27,6 +27,10 @@
       </ros>
       <link_name>gripper_grasp_link</link_name>
-      <max_distance>0.08</max_distance>
+      <max_distance>0.15</max_distance>
       <fixed>ground_plane</fixed>
+      <fixed>table_in</fixed>
+      <fixed>table_out</fixed>
+      <fixed>station_tray_in</fixed>
+      <fixed>station_tray_out</fixed>
       <fixed>rack_a_level_1_plank</fixed>
       <fixed>rack_a_level_2_plank</fixed>
@@ -35,4 +39,14 @@
       <fixed>shelf_tray_0</fixed>
       <fixed>shelf_tray_1</fixed>
+      <fixed>shelf_tray_2</fixed>
+      <fixed>shelf_tray_3</fixed>
+      <fixed>shelf_tray_4</fixed>
+      <fixed>shelf_tray_5</fixed>
+      <fixed>shelf_tray_6</fixed>
+      <fixed>shelf_tray_7</fixed>
+      <fixed>shelf_tray_8</fixed>
+      <fixed>shelf_tray_9</fixed>
+      <fixed>shelf_tray_10</fixed>
+      <fixed>shelf_tray_11</fixed>
     </plugin>
   </gazebo>

File: src/wh_description/urdf/ros2_control.xacro (robot description, xacro)
@@ -34,4 +34,18 @@
       <state_interface name="velocity"/>
     </joint>
+    <joint name="left_finger_joint">
+      <command_interface name="position"/>
+      <state_interface name="position">
+        <param name="initial_value">0.0</param>
+      </state_interface>
+      <state_interface name="velocity"/>
+    </joint>
+    <joint name="right_finger_joint">
+      <command_interface name="position"/>
+      <state_interface name="position">
+        <param name="initial_value">0.0</param>
+      </state_interface>
+      <state_interface name="velocity"/>
+    </joint>
   </ros2_control>
   <gazebo>

File: src/wh_description/urdf/sensors.xacro (robot description, xacro)
@@ -205,34 +205,34 @@
   <!-- ======================================================== -->
   <!-- ======================================================== -->
-  <!-- HAND CAMERA (Gắn trên đế tay kẹp bẻ ngang, nhìn về phía trước) -->
+  <!-- HAND CAMERA (Gắn trên sống lưng cụm tay kẹp, nhìn xuống hộp) -->
   <!-- ======================================================== -->
   <joint name="hand_camera_joint" type="fixed">
     <parent link="tool_link"/>
     <child link="hand_camera_link"/>
-    <!-- Gắn trên sống lưng khớp bẻ ngang, nhìn theo phương +X và chúi nhẹ 12.6 độ xuống hộp -->
-    <origin xyz="0.006 0.0 -0.038" rpy="0 0.22 0"/>
+    <!-- Gắn chuẩn trên sống lưng mặt bích kẹp (x=0.016m, z=-0.020m), hướng thẳng tâm và chúc 50 độ (0.87 rad) xuống tâm hộp giữa 2 má kẹp -->
+    <origin xyz="0.016 0.0 -0.020" rpy="0 0.87 0"/>
   </joint>
   <link name="hand_camera_link">
-    <!-- Ngàm đỡ bắt bulông vào mặt sau đế tay kẹp (nằm phía sau sensor) -->
-    <visual>
-      <origin xyz="-0.015 0 0" rpy="0 0 0"/>
-      <geometry>
-        <box size="0.016 0.032 0.016"/>
+    <!-- Ngàm đỡ bắt bulông vào mặt trên đế kẹp (bracket) -->
+    <visual>
+      <origin xyz="-0.008 0 0" rpy="0 0 0"/>
+      <geometry>
+        <box size="0.012 0.026 0.012"/>
       </geometry>
       <material name="cam_bracket"/>
     </visual>
-    <!-- Thân vỏ camera (nằm phía sau sensor) -->
-    <visual>
-      <origin xyz="-0.005 0 0" rpy="0 0 0"/>
-      <geometry>
-        <box size="0.020 0.036 0.020"/>
+    <!-- Thân vỏ camera gọn gàng (housing) -->
+    <visual>
+      <origin xyz="0 0 0" rpy="0 0 0"/>
+      <geometry>
+        <box size="0.016 0.028 0.018"/>
       </geometry>
       <material name="cam_body"/>
     </visual>
-    <!-- Ống kính nhìn thẳng theo trục quang học -->
-    <visual>
-      <origin xyz="0.005 0 0" rpy="0 1.57079632679 0"/>
-      <geometry>
-        <cylinder radius="0.007" length="0.006"/>
+    <!-- Ống kính nhìn thẳng theo trục quang học hướng vào tâm kẹp -->
+    <visual>
+      <origin xyz="0.009 0 0" rpy="0 1.57079632679 0"/>
+      <geometry>
+        <cylinder radius="0.006" length="0.006"/>
       </geometry>
       <material name="cam_lens"/>
